Commit message: 仿真增加底盘移动部分, 发布/cmd_vel topic用于移动底盘

File: src/R2_description/urdf/R2.xacro (robot description, xacro)
@@ -3,5 +3,5 @@
 <!-- <xacro:include filename="$(find ros2_livox_simulation)/urdf/mid360.xacro" /> -->
 <xacro:include filename="$(find r2_description)/urdf/materials.xacro" />
-<xacro:include filename="$(find r2_description)/urdf/R2.trans" />
+<!-- <xacro:include filename="$(find r2_description)/urdf/R2.trans" /> -->
 <xacro:include filename="$(find r2_description)/urdf/R2.gazebo" />
 <link name="base_link">
@@ -39,7 +39,7 @@
   </visual>
   <collision>
-    <origin xyz="-0.225 0.27 -0.01" rpy="0 0 0"/>
+    <origin xyz="0 0 0" rpy="1.570796 0 0"/>
     <geometry>
-      <mesh filename="file://$(find r2_description)/meshes/wheel_1_1.stl" scale="0.001 0.001 0.001"/>
+      <cylinder radius="0.06" length="0.06"/>
     </geometry>
   </collision>
@@ -59,7 +59,7 @@
   </visual>
   <collision>
-    <origin xyz="0.225 0.27 -0.01" rpy="0 0 0"/>
+    <origin xyz="0 0 0" rpy="1.570796 0 0"/>
     <geometry>
-      <mesh filename="file://$(find r2_description)/meshes/wheel_2_1.stl" scale="0.001 0.001 0.001"/>
+      <cylinder radius="0.06" length="0.06"/>
     </geometry>
   </collision>
@@ -79,7 +79,7 @@
   </visual>
   <collision>
-    <origin xyz="0.225 -0.27 -0.01" rpy="0 0 0"/>
+    <origin xyz="0 0 0" rpy="1.570796 0 0"/>
     <geometry>
-      <mesh filename="file://$(find r2_description)/meshes/wheel_3_1.stl" scale="0.001 0.001 0.001"/>
+      <cylinder radius="0.06" length="0.06"/>
     </geometry>
   </collision>
@@ -99,127 +99,7 @@
   </visual>
   <collision>
-    <origin xyz="-0.225 -0.27 -0.01" rpy="0 0 0"/>
+    <origin xyz="0 0 0" rpy="1.570796 0 0"/>
     <geometry>
-      <mesh filename="file://$(find r2_description)/meshes/wheel_4_1.stl" scale="0.001 0.001 0.001"/>
-    </geometry>
-  </collision>
-</link>
-<link name="rise_link_1">
-  <inertial>
-    <origin xyz="-0.00999999999997675 -0.009665452061459481 0.015000000000000006" rpy="0 0 0"/>
-    <mass value="0.5"/>
-    <inertia ixx="0.001" iyy="0.001" izz="0.001" ixy="0.0" iyz="0.0" ixz="0.0"/>
-  </inertial>
-  <visual>
-    <origin xyz="-0.284 -0.08 -0.055" rpy="0 0 0"/>
-    <geometry>
-      <mesh filename="file://$(find r2_description)/meshes/rise_link_1.stl" scale="0.001 0.001 0.001"/>
-    </geometry>
-    <material name="silver"/>
-  </visual>
-  <collision>
-    <origin xyz="0 0 0" rpy="0 0 0"/>
-    <geometry>
-      <box size="0.01 0.01 0.01"/>
-    </geometry>
-  </collision>
-</link>
-<link name="big_arm_1">
-  <inertial>
-    <origin xyz="0.04808967127134256 -0.049999999999999926 4.163336342344337e-17" rpy="0 0 0"/>
-    <mass value="6.600509248834649"/>
-    <inertia ixx="0.01805" iyy="0.039183" izz="0.039158" ixy="0.0" iyz="0.0" ixz="0.0"/>
-  </inertial>
-  <visual>
-    <origin xyz="-0.274 -0.05 -0.07" rpy="0 0 0"/>
-    <geometry>
-      <mesh filename="file://$(find r2_description)/meshes/big_arm_1.stl" scale="0.001 0.001 0.001"/>
-    </geometry>
-    <material name="silver"/>
-  </visual>
-  <collision>
-    <origin xyz="-0.274 -0.05 -0.07" rpy="0 0 0"/>
-    <geometry>
-      <mesh filename="file://$(find r2_description)/meshes/big_arm_1.stl" scale="0.001 0.001 0.001"/>
-    </geometry>
-  </collision>
-</link>
-<link name="small_arm_1">
-  <inertial>
-    <origin xyz="-0.05476973272585678 -0.03999999999999998 0.04000000000000001" rpy="0 0 0"/>
-    <mass value="3.6300692488346558"/>
-    <inertia ixx="0.00598" iyy="0.012616" izz="0.013128" ixy="-0.0" iyz="0.0" ixz="0.0"/>
-  </inertial>
-  <visual>
-    <origin xyz="-0.439 -0.04 -0.03" rpy="0 0 0"/>
-    <geometry>
-      <mesh filename="file://$(find r2_description)/meshes/small_arm_1.stl" scale="0.001 0.001 0.001"/>
-    </geometry>
-    <material name="silver"/>
-  </visual>
-  <collision>
-    <origin xyz="-0.439 -0.04 -0.03" rpy="0 0 0"/>
-    <geometry>
-      <mesh filename="file://$(find r2_description)/meshes/small_arm_1.stl" scale="0.001 0.001 0.001"/>
-    </geometry>
-  </collision>
-</link>
-<link name="head_link_1">
-  <inertial>
-    <origin xyz="0.05282614697034416 -0.03 0.0" rpy="0 0 0"/>
-    <mass value="4.263104309432333"/>
-    <inertia ixx="0.002519" iyy="0.009527" izz="0.009566" ixy="0.0" iyz="-0.0" ixz="0.0"/>
-  </inertial>
-  <visual>
-    <origin xyz="-0.469 -0.03 -0.07" rpy="0 0 0"/>
-    <geometry>
-      <mesh filename="file://$(find r2_description)/meshes/head_link_1.stl" scale="0.001 0.001 0.001"/>
-    </geometry>
-    <material name="silver"/>
-  </visual>
-  <collision>
-    <origin xyz="-0.469 -0.03 -0.07" rpy="0 0 0"/>
-    <geometry>
-      <mesh filename="file://$(find r2_description)/meshes/head_link_1.stl" scale="0.001 0.001 0.001"/>
-    </geometry>
-  </collision>
-</link>
-<link name="y_move_1">
-  <inertial>
-    <origin xyz="-0.02000000000000013 -0.01999999999999998 0.097" rpy="0 0 0"/>
-    <mass value="2.43664"/>
-    <inertia ixx="0.007967" iyy="0.007967" izz="0.00065" ixy="0.0" iyz="0.0" ixz="0.0"/>
-  </inertial>
-  <visual>
-    <origin xyz="-0.205 -0.05 -0.02" rpy="0 0 0"/>
-    <geometry>
-      <mesh filename="file://$(find r2_description)/meshes/y_move_1.stl" scale="0.001 0.001 0.001"/>
-    </geometry>
-    <material name="silver"/>
-  </visual>
-  <collision>
-    <origin xyz="0 0 0" rpy="0 0 0"/>
-    <geometry>
-      <box size="0.01 0.01 0.01"/>
-    </geometry>
-  </collision>
-</link>
-<link name="x_move_1">
-  <inertial>
-    <origin xyz="0.01999999999999988 -0.009999999999999983 -0.009999999999999926" rpy="0 0 0"/>
-    <mass value="0.5"/>
-    <inertia ixx="0.001" iyy="0.001" izz="0.001" ixy="0.0" iyz="-0.0" ixz="0.0"/>
-  </inertial>
-  <visual>
-    <origin xyz="-0.165 -0.01 -0.214" rpy="0 0 0"/>
-    <geometry>
-      <mesh filename="file://$(find r2_description)/meshes/x_move_1.stl" scale="0.001 0.001 0.001"/>
-    </geometry>
-    <material name="silver"/>
-  </visual>
-  <collision>
-    <origin xyz="0 0 0" rpy="0 0 0"/>
-    <geometry>
-      <box size="0.01 0.01 0.01"/>
+      <cylinder radius="0.06" length="0.06"/>
     </geometry>
   </collision>
@@ -253,4 +133,5 @@
   <child link="wheel_1_1"/>
   <axis xyz="0.0 1.0 0.0"/>
+  <dynamics damping="1.0" friction="1.0"/>
 </joint>
 <joint name="spin_2" type="continuous">
@@ -259,4 +140,5 @@
   <child link="wheel_2_1"/>
   <axis xyz="0.0 1.0 0.0"/>
+  <dynamics damping="1.0" friction="1.0"/>
 </joint>
 <joint name="spin_3" type="continuous">
@@ -264,5 +146,6 @@
   <parent link="base_link"/>
   <child link="wheel_3_1"/>
-  <axis xyz="0.0 -1.0 0.0"/>
+  <axis xyz="0.0 1.0 0.0"/>
+  <dynamics damping="1.0" friction="1.0"/>
 </joint>
 <joint name="spin_4" type="continuous">
@@ -270,49 +153,6 @@
   <parent link="base_link"/>
   <child link="wheel_4_1"/>
-  <axis xyz="0.0 -1.0 0.0"/>
-</joint>
-<joint name="slide_5" type="prismatic">
-  <origin xyz="0.284 0.08 0.055" rpy="0 0 0"/>
-  <parent link="base_link"/>
-  <child link="rise_link_1"/>
-  <axis xyz="0.0 0.0 1.0"/>
-  <dynamics damping="10.0" friction="1.0"/>
-  <limit upper="0.617" lower="0.0" effort="100" velocity="100"/>
-</joint>
-<joint name="spin_6" type="continuous">
-  <origin xyz="-0.01 -0.03 0.015" rpy="0 0 0"/>
-  <parent link="rise_link_1"/>
-  <child link="big_arm_1"/>
   <axis xyz="0.0 1.0 0.0"/>
-</joint>
-<joint name="slide_7" type="prismatic">
-  <origin xyz="0.165 -0.01 -0.04" rpy="0 0 0"/>
-  <parent link="big_arm_1"/>
-  <child link="small_arm_1"/>
-  <axis xyz="1.0 0.0 0.0"/>
-  <dynamics damping="10.0" friction="1.0"/>
-  <limit upper="0.555" lower="0.0" effort="100" velocity="100"/>
-</joint>
-<joint name="spin_8" type="continuous">
-  <origin xyz="0.03 -0.01 0.04" rpy="0 0 0"/>
-  <parent link="small_arm_1"/>
-  <child link="head_link_1"/>
-  <axis xyz="0.0 -1.0 0.0"/>
-</joint>
-<joint name="slide_9" type="prismatic">
-  <origin xyz="-0.069 0.0 -0.05" rpy="0 0 0"/>
-  <parent link="big_arm_1"/>
-  <child link="y_move_1"/>
-  <axis xyz="0.0 1.0 0.0"/>
-  <dynamics damping="10.0" friction="1.0"/>
-  <limit upper="0.1" lower="0.0" effort="100" velocity="100"/>
-</joint>
-<joint name="slide_10" type="prismatic">
-  <origin xyz="-0.04 -0.04 0.194" rpy="0 0 0"/>
-  <parent link="y_move_1"/>
-  <child link="x_move_1"/>
-  <axis xyz="0.0 0.0 1.0"/>
-  <dynamics damping="10.0" friction="1.0"/>
-  <limit upper="0.1" lower="0.0" effort="100" velocity="100"/>
+  <dynamics damping="1.0" friction="1.0"/>
 </joint>
 <joint name="slide_11" type="fixed">

Commit message: 加入摄像头

File: src/R2_description/urdf/R2.xacro (robot description, xacro)
@@ -128,4 +128,28 @@
     <origin xyz="0 0 0.025" rpy="0 0 0"/>
 </xacro:mid360>
+<link name="camera_link">
+  <visual>
+    <origin xyz="0 0 0" rpy="0 0 0" />
+    <geometry>
+      <box size="0.025 0.09 0.025" />
+    </geometry>
+    <material name="black" />
+  </visual>
+  <collision>
+    <origin xyz="0 0 0" rpy="0 0 0" />
+    <geometry>
+      <box size="0.025 0.09 0.025" />
+    </geometry>
+  </collision>
+  <inertial>
+    <mass value="0.072" />
+    <inertia ixx="0.001" ixy="0" ixz="0" iyy="0.001" iyz="0" izz="0.001" />
+  </inertial>
+</link>
+<joint name="camera_joint" type="fixed">
+  <parent link="base_link" />
+  <child link="camera_link" />
+  <origin xyz="0.90 0 0.60" rpy="0 1.5708 0" />
+</joint>
 <joint name="spin_1" type="continuous">
   <origin xyz="0.225 -0.27 0.01" rpy="0 0 0"/>
