Commit message: 修复bug, 完成fast-lio2测试, 后续再加上nav2测试

File: src/R2_description/urdf/R2.xacro (robot description, xacro)
@@ -126,5 +126,5 @@
 </link>
 <xacro:mid360 name="livox" parent="mid360_1" topic="/livox/lidar">
-    <origin xyz="0 0 0.025" rpy="0 0 0"/>
+    <origin xyz="0 0 0" rpy="0 0 0"/>
 </xacro:mid360>
 <link name="camera_link">
@@ -150,5 +150,5 @@
   <parent link="base_link" />
   <child link="camera_link" />
-  <origin xyz="0.90 0 0.60" rpy="0 1.5708 0" />
+  <origin xyz="0.5 0 0.50" rpy="0 1.5708 0" />
 </joint>
 <joint name="spin_1" type="continuous">
